File: PCB/termocuplaJ/termocuplaJ.sch (KiCad schematic (older format))
At the start: 38 parts, among them J1 Screw_Terminal_01x02, J10 Keypad4x4, J11 SPI, J2 Screw_Terminal_01x02, J3 Screw_Terminal_01x02, J4 2-relay-module, J5 J-THERMO, J6 Conn_01x04_Male, J7 Keypad4x4, J8 Conn_01x05_Male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

Commit message: To release!
Parts:
- added C5: 100uF/16V, Capacitor_THT:CP_Radial_D5.0mm_P2.00mm, symbol Device:CP1_Small
- added D4, D5, D6, D7: 1N4148, Diode_THT:D_DO-35_SOD27_P7.62mm_Horizontal, symbol Diode:1N4148
- added D8: LED-ACT, symbol Device:LED
- added R9: 10k, Resistor_THT:R_Axial_DIN0207_L6.3mm_D2.5mm_P10.16mm_Horizontal, symbol Device:R
- J1: value Screw_Terminal_01x02 -> POWER INPUT 24VDC
- J2: value Screw_Terminal_01x02 -> PULSE 24V-NEWPIECE
- J3: value Screw_Terminal_01x02 -> PULSE 24V-RESET
- gave numbers to parts that had none: 1
Connections:
- net labels added: FIL1k, FIL2k, FIL3k, FIL4k
- wire segments 171 -> 192
Other:
- note added: "RELAY2: CTRL TEMP \nPID OUTPUT\n"
- moved on the sheet: D2, D3, H1, H3, H5, H7, J10, J2, J3, J4, J7, R3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
